File: ESP32_Shield.kicad_pcb (KiCad board)
At the start: 4 copper layers, 69 x 40.6 mm, 42 parts, among them J1 BME280, SHT40 Module, J10 SCD40 Module, J11 Conn_01x03, J12 Conn_01x03, J13 SCD40 Module, J14 BME280, SHT40 Module, J15 mmWave Connector, J16 mmWave Connector, J17 mmWave Connector, J2 SCD40 Module, J3 Conn_01x02, J4 Qwiic_Vertical, J5 Conn_01x02, J6 Conn_01x02, J7 Conn_01x03, J8 Conn_01x03, J9 VL53L0X Module, Q1 PT19-21C, U5 TLP175A

Commit message: Add project-local KiCad libraries
Parts:
- U1: footprint ThomasFootprints:ESP32_S3_zeroBoard -> ESP32_Shield_Custom_Footprints:ESP32-S3-Zero
- U2: footprint LibraryThomas:Unbenannt -> ESP32_Shield_Sensor_Footprints:HLK-LD2410B-mmWave-Sensor
- U4: footprint LibraryThomas:PIR_SR602 -> ESP32_Shield_Sensor_Footprints:SR602-PIR-Motion-Sensor
Changed lines of the file:
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@@
 		)
 	)
-	(footprint "LibraryThomas:PIR_SR602"
+	(footprint "ESP32_Shield_Sensor_Footprints:SR602-PIR-Motion-Sensor"
 		(layer "F.Cu")
 		(at 132 93.58)
@@
 		)
 	)
-	(footprint "LibraryThomas:Unbenannt"
+	(footprint "ESP32_Shield_Sensor_Footprints:HLK-LD2410B-mmWave-Sensor"
 		(layer "F.Cu")
 		(at 100.5 72.25)
@@
 		)
 	)
-	(footprint "ThomasFootprints:ESP32_S3_zeroBoard"
+	(footprint "ESP32_Shield_Custom_Footprints:ESP32-S3-Zero"
 		(layer "F.Cu")
 		(at 118.87 83.42 90)
