File: ESP32_Shield.kicad_sch (KiCad schematic)
At the start: 42 parts, among them J1 BME280, SHT40 Module, J10 SCD40 Module, J11 Conn_01x03, J12 Conn_01x03, J13 SCD40 Module, J14 BME280, SHT40 Module, J15 mmWave Connector, J16 mmWave Connector, J17 mmWave Connector, J2 SCD40 Module, J3 Conn_01x02, J4 Qwiic_Vertical, J5 Conn_01x02, J6 Conn_01x02, J7 Conn_01x03, J8 Conn_01x03, J9 VL53L0X Module, Q1 PT19-21C, U5 TLP175A

Commit message: Upgrade project files to KiCad 10
Parts:
- U1, U2, U4: value ~ -> (none)

Commit message: Add project-local KiCad libraries
Parts:
- U1: footprint ThomasFootprints:ESP32_S3_zeroBoard -> ESP32_Shield_Custom_Footprints:ESP32-S3-Zero; symbol ThomasPersolLib:ESP32-S3_zersoBoard -> ESP32_Shield_Custom_Symbols:ESP32-S3-Zero
- U2: footprint LibraryThomas:Unbenannt -> ESP32_Shield_Sensor_Footprints:HLK-LD2410B-mmWave-Sensor; symbol SymbolThomas:U1 -> ESP32_Shield_Sensor_Symbols:HLK-LD2410B-mmWave-Sensor
- U4: footprint LibraryThomas:PIR_SR602 -> ESP32_Shield_Sensor_Footprints:SR602-PIR-Motion-Sensor; symbol SymbolThomas:PIR_SR602 -> ESP32_Shield_Sensor_Symbols:SR602-PIR-Motion-Sensor
Changed lines of the file:
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@@
 	)
 	(symbol
-		(lib_id "ThomasPersolLib:ESP32-S3_zersoBoard")
+		(lib_id "ESP32_Shield_Custom_Symbols:ESP32-S3-Zero")
 		(at 119.38 66.04 0)
 		(unit 1)
@@
 			)
 		)
-		(property "Footprint" "ThomasFootprints:ESP32_S3_zeroBoard"
+		(property "Footprint" "ESP32_Shield_Custom_Footprints:ESP32-S3-Zero"
 			(at 119.38 66.04 0)
 			(hide yes)
@@
 	)
 	(symbol
-		(lib_id "SymbolThomas:U1")
+		(lib_id "ESP32_Shield_Sensor_Symbols:HLK-LD2410B-mmWave-Sensor")
 		(at 189.23 143.51 0)
 		(unit 1)
@@
 			)
 		)
-		(property "Footprint" "LibraryThomas:Unbenannt"
+		(property "Footprint" "ESP32_Shield_Sensor_Footprints:HLK-LD2410B-mmWave-Sensor"
 			(at 189.23 143.51 0)
 			(hide yes)
@@
 	)
 	(symbol
-		(lib_id "SymbolThomas:PIR_SR602")
+		(lib_id "ESP32_Shield_Sensor_Symbols:SR602-PIR-Motion-Sensor")
 		(at 128.27 21.59 0)
 		(unit 1)
@@
 			)
 		)
-		(property "Footprint" "LibraryThomas:PIR_SR602"
+		(property "Footprint" "ESP32_Shield_Sensor_Footprints:SR602-PIR-Motion-Sensor"
 			(at 128.27 21.59 0)
 			(hide yes)
